File: Hardware/BC118_Mate.brd (EAGLE design)
At the start: 25.4 x 47 mm, 27 parts, among them Q1 BSS138, U2 AP2202-ADJ

Commit message: V01 ready for protos
Parts:
- added JP4: (no value), SparkFun-Connectors:1X06
Connections:
- new net CTS: JP1.CTS, JP4.CTS
- new net DTR: JP1.DTR, JP4.DTR
- net GND: now also JP4.GND
- net RXI: now also JP4.RXI
- net TXO: now also JP4.TXO
- net VIN: now also JP4.VCC
Routing:
- net TXO: track 30.4 -> 33.0 mm
- net DTR: track 0.00 -> 2.54 mm
- net CTS: track 0.00 -> 2.54 mm
- net VIN: track 23.0 -> 25.5 mm
- net RXI: track 11.3 -> 13.8 mm
Other:
- board size 25.4 x 47 mm -> 25.4 x 49.5 mm
- board text added: "BLK"
- board text added: "GRN"
Changed lines of the file:
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@@
 <grid distance="0.05" unitdist="inch" unit="inch" style="lines" multiple="1" display="yes" altdistance="0.005" altunitdist="inch" altunit="inch"/>
 <layers>
-<layer number="1" name="Top" color="4" fill="1" visible="no" active="yes"/>
+<layer number="1" name="Top" color="4" fill="1" visible="yes" active="yes"/>
 <layer number="2" name="Route2" color="1" fill="3" visible="no" active="yes"/>
 <layer number="15" name="Route15" color="4" fill="6" visible="no" active="yes"/>
@@
 <layer number="19" name="Unrouted" color="6" fill="1" visible="yes" active="yes"/>
 <layer number="20" name="Dimension" color="15" fill="1" visible="yes" active="yes"/>
-<layer number="21" name="tPlace" color="16" fill="1" visible="no" active="yes"/>
+<layer number="21" name="tPlace" color="16" fill="1" visible="yes" active="yes"/>
 <layer number="22" name="bPlace" color="14" fill="1" visible="yes" active="yes"/>
-<layer number="23" name="tOrigins" color="15" fill="1" visible="no" active="yes"/>
+<layer number="23" name="tOrigins" color="15" fill="1" visible="yes" active="yes"/>
 <layer number="24" name="bOrigins" color="15" fill="1" visible="yes" active="yes"/>
 <layer number="25" name="tNames" color="7" fill="1" visible="no" active="yes"/>
@@
 <layer number="43" name="vRestrict" color="2" fill="10" visible="no" active="yes"/>
 <layer number="44" name="Drills" color="7" fill="1" visible="no" active="yes"/>
-<layer number="45" name="Holes" color="7" fill="1" visible="no" active="yes"/>
+<layer number="45" name="Holes" color="7" fill="1" visible="yes" active="yes"/>
 <layer number="46" name="Milling" color="3" fill="1" visible="no" active="yes"/>
-<layer number="51" name="tDocu" color="6" fill="1" visible="no" active="yes"/>
+<layer number="51" name="tDocu" color="6" fill="1" visible="yes" active="yes"/>
 <layer number="52" name="bDocu" color="7" fill="1" visible="no" active="yes"/>
 <layer number="3" name="Route3" color="4" fill="3" visible="no" active="no"/>
@@
 <text x="13.97" y="-0.889" size="1.778" layer="22" font="vector" ratio="15" rot="MR90" align="center-left">DTR</text>
 <wire x1="-5.08" y1="43.18" x2="20.32" y2="43.18" width="0.1524" layer="20"/>
-<wire x1="20.32" y1="43.18" x2="20.32" y2="-3.81" width="0.1524" layer="20"/>
-<wire x1="20.32" y1="-3.81" x2="-5.08" y2="-3.81" width="0.1524" layer="20"/>
-<wire x1="-5.08" y1="43.18" x2="-5.08" y2="-3.81" width="0.1524" layer="20"/>
+<wire x1="20.32" y1="43.18" x2="20.32" y2="-6.35" width="0.1524" layer="20"/>
+<wire x1="20.32" y1="-6.35" x2="-5.08" y2="-6.35" width="0.1524" layer="20"/>
+<wire x1="-5.08" y1="43.18" x2="-5.08" y2="-6.35" width="0.1524" layer="20"/>
 <text x="-2.159" y="29.21" size="1.016" layer="21" font="vector" ratio="15" rot="R90" align="top-center">A2</text>
 <text x="-2.159" y="26.67" size="1.016" layer="21" font="vector" ratio="15" rot="R90" align="top-center">A1</text>
@@
 <text x="-2.032" y="16.51" size="1.016" layer="21" font="vector" ratio="15" rot="R90" align="top-center">P8</text>
 <text x="-2.032" y="13.97" size="1.016" layer="21" font="vector" ratio="15" rot="R90" align="top-center">WK</text>
-<text x="-2.032" y="11.43" size="1.016" layer="21" font="vector" ratio="15" rot="R90" align="top-center">VIN</text>
-<text x="-2.032" y="8.89" size="1.016" layer="21" font="vector" ratio="15" rot="R90" align="top-center">GND</text>
+<text x="-2.032" y="11.43" size="0.8128" layer="21" font="vector" ratio="15" rot="R90" align="top-center">VIN</text>
+<text x="-2.032" y="8.89" size="0.8128" layer="21" font="vector" ratio="15" rot="R90" align="top-center">GND</text>
 <text x="17.399" y="29.21" size="1.016" layer="21" font="vector" ratio="15" rot="R90" align="bottom-center">P5</text>
 <text x="17.399" y="26.67" size="1.016" layer="21" font="vector" ratio="15" rot="R90" align="bottom-center">P6</text>
@@
 <text x="17.399" y="16.51" size="1.016" layer="21" font="vector" ratio="15" rot="R90" align="bottom-center">P10</text>
 <text x="17.399" y="13.97" size="1.016" layer="21" font="vector" ratio="15" rot="R90" align="bottom-center">P2</text>
-<text x="17.399" y="11.43" size="1.016" layer="21" font="vector" ratio="15" rot="R90" align="bottom-center">VDD</text>
-<text x="17.399" y="8.763" size="1.016" layer="21" font="vector" ratio="15" rot="R90" align="bottom-center">GND</text>
+<text x="17.399" y="11.43" size="0.8128" layer="21" font="vector" ratio="15" rot="R90" align="bottom-center">VDD</text>
+<text x="17.399" y="8.763" size="0.8128" layer="21" font="vector" ratio="15" rot="R90" align="bottom-center">GND</text>
 <text x="10.287" y="11.684" size="1.016" layer="21" font="vector" ratio="15" align="bottom-center">LEDS</text>
 <text x="1.397" y="5.08" size="1.016" layer="21" font="vector" ratio="15" rot="R180" align="bottom-center">INP</text>
@@
 <text x="17.78" y="16.51" size="1.016" layer="22" font="vector" ratio="15" rot="MR90" align="top-center">P10</text>
 <text x="17.78" y="13.97" size="1.016" layer="22" font="vector" ratio="15" rot="MR90" align="top-center">P2</text>
-<text x="17.78" y="11.43" size="1.016" layer="22" font="vector" ratio="15" rot="MR90" align="top-center">VDD</text>
-<text x="17.78" y="8.763" size="1.016" layer="22" font="vector" ratio="15" rot="MR90" align="top-center">GND</text>
+<text x="17.78" y="11.43" size="0.8128" layer="22" font="vector" ratio="15" rot="MR90" align="top-center">VDD</text>
+<text x="17.78" y="8.763" size="0.8128" layer="22" font="vector" ratio="15" rot="MR90" align="top-center">GND</text>
 <text x="10.287" y="5.461" size="1.4224" layer="22" font="vector" ratio="15" rot="MR0" align="bottom-center">BLE Mate</text>
 <text x="-2.413" y="29.21" size="1.016" layer="22" font="vector" ratio="15" rot="MR90" align="bottom-center">A2</text>
@@
 <text x="-2.54" y="16.51" size="1.016" layer="22" font="vector" ratio="15" rot="MR90" align="bottom-center">P8</text>
 <text x="-2.54" y="13.97" size="1.016" layer="22" font="vector" ratio="15" rot="MR90" align="bottom-center">WK</text>
-<text x="-2.54" y="11.43" size="1.016" layer="22" font="vector" ratio="15" rot="MR90" align="bottom-center">VIN</text>
-<text x="-2.54" y="8.89" size="1.016" layer="22" font="vector" ratio="15" rot="MR90" align="bottom-center">GND</text>
+<text x="-2.54" y="11.43" size="0.8128" layer="22" font="vector" ratio="15" rot="MR90" align="bottom-center">VIN</text>
+<text x="-2.54" y="8.89" size="0.8128" layer="22" font="vector" ratio="15" rot="MR90" align="bottom-center">GND</text>
+<text x="-0.254" y="-5.334" size="1.27" layer="21" font="vector" ratio="15" rot="R90">BLK</text>
+<text x="16.764" y="-5.461" size="1.27" layer="21" font="vector" ratio="15" rot="R90">GRN</text>
+<text x="15.494" y="-5.461" size="1.27" layer="22" font="vector" ratio="15" rot="MR90">GRN</text>
+<text x="-1.524" y="-5.334" size="1.27" layer="22" font="vector" ratio="15" rot="MR90">BLK</text>
 </plain>
 <attributes>
@@
 <element name="LOGO3" library="SparkFun-Aesthetics" package="SFE_LOGO_NAME_.1" value="SFE_LOGO_NAME.1_INCH" x="11.557" y="32.512" rot="MR0"/>
 <element name="LOGO4" library="SparkFun-Aesthetics" package="OSHW-LOGO-S" value="OSHW-LOGOS" x="-2.159" y="33.02" rot="MR0"/>
+<element name="JP4" library="SparkFun-Connectors" package="1X06" value="" x="13.97" y="-5.08" rot="R180"/>
 </elements>
 <signals>
@@
 <wire x1="10.16" y1="4.064" x2="8.89" y2="2.794" width="0.254" layer="1"/>
 <wire x1="8.89" y1="2.794" x2="8.89" y2="-2.54" width="0.254" layer="1"/>
+<contactref element="JP4" pad="TXO"/>
+<wire x1="8.89" y1="-2.54" x2="8.89" y2="-5.08" width="0.254" layer="16"/>
 </signal>
 <signal name="RXI">
@@
 <wire x1="14.732" y1="3.81" x2="15.113" y2="4.191" width="0.254" layer="1"/>
 <wire x1="15.113" y1="4.191" x2="15.113" y2="5.5" width="0.254" layer="1"/>
+<contactref element="JP4" pad="RXI"/>
+<wire x1="11.43" y1="-2.54" x2="11.43" y2="-5.08" width="0.254" layer="16"/>
 </signal>
 <signal name="N$3">
@@
 <vertex x="-5.08" y="38.1"/>
 <vertex x="20.32" y="38.1"/>
-<vertex x="20.32" y="-3.81"/>
-<vertex x="-5.08" y="-3.81"/>
+<vertex x="20.32" y="-6.35"/>
+<vertex x="-5.08" y="-6.35"/>
 </polygon>
 <polygon width="0.254" layer="16" isolate="0.3048">
 <vertex x="-5.08" y="38.1"/>
 <vertex x="20.32" y="38.1"/>
-<vertex x="20.32" y="-3.81"/>
-<vertex x="-5.08" y="-3.81"/>
+<vertex x="20.32" y="-6.35"/>
+<vertex x="-5.08" y="-6.35"/>
 </polygon>
 <via x="0" y="21.717" extent="1-16" drill="0.508"/>
@@
 <via x="0" y="8.128" extent="1-16" drill="0.508"/>
 <via x="-0.889" y="4.445" extent="1-16" drill="0.508"/>
+<contactref element="JP4" pad="GND"/>
 </signal>
 <signal name="VDD">
@@
 <wire x1="5.842" y1="3.683" x2="6.35" y2="3.175" width="0.254" layer="1"/>
 <wire x1="6.35" y1="3.175" x2="6.35" y2="-2.54" width="0.254" layer="1"/>
+<contactref element="JP4" pad="VCC"/>
+<wire x1="6.35" y1="-2.54" x2="6.35" y2="-5.08" width="0.254" layer="16"/>
 </signal>
 <signal name="N$4">
@@
 <wire x1="-2.667" y1="16.51" x2="-3.81" y2="16.51" width="0.254" layer="1"/>
 </signal>
+<signal name="DTR">
+<contactref element="JP1" pad="DTR"/>
+<contactref element="JP4" pad="DTR"/>
+<wire x1="13.97" y1="-2.54" x2="13.97" y2="-5.08" width="0.254" layer="16"/>
+</signal>
+<signal name="CTS">
+<contactref element="JP1" pad="CTS"/>
+<contactref element="JP4" pad="CTS"/>
+<wire x1="3.81" y1="-2.54" x2="3.81" y2="-5.08" width="0.254" layer="16"/>
+</signal>
 </signals>
