File: Hardware/BC118_Mate.brd (EAGLE design)
At the start: 25.4 x 49.5 mm, 28 parts, among them Q1 BSS138, U2 AP2202-ADJ

Commit message: Change LED pin assignments to match new firmware
Parts:
- LED0: value RED -> BLUE
- LED1: value BLUE -> RED
- moved LED0 3.05 mm to (8.64, 19.9)
- moved LED1 3.05 mm to (11.7, 19.9)
Connections:
- net N$8: now also LED0.C; no longer LED1.C
- net N$9: now also LED1.C; no longer LED0.C
- net PIO_10: no longer LED1.A
- net PIO_4: now also LED0.A
- net PIO_9: now also LED1.A; no longer LED0.A
Routing:
- net PIO_4: track 15.4 -> 26.3 mm, vias 2 -> 4
- net PIO_10: track 27.9 -> 25.1 mm, vias 2 -> 1
- net WAKE: track 36.5 -> 37.3 mm
- net PIO_8: track 18.8 -> 19.5 mm
Other:
- board text added: "V10"
- board text removed: "V01"

Commit message: Ready for reds
Parts:
- LOGO3: value SFE_LOGO_NAME.1_INCH -> SFE_LOGO_NAME_FLAME.1_INCH; device SparkFun-Aesthetics:SFE_LOGO_NAME_.1 -> SparkFun-Aesthetics:SFE_LOGO_NAME_FLAME_.1
- R6: value 26.7k -> 16.2k
- R7: value 16.2k -> 26.7k
- moved LOGO3 0.85 mm to (12.3, 32.9)
- moved LOGO1 0.46 mm to (20.6, -4.19)
Other:
- board text added: "BLE Mate2"
- board text removed: "BLE Mate"
Changed lines of the file:
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@@
 <text x="1.397" y="5.08" size="1.016" layer="21" font="vector" ratio="15" rot="R180" align="bottom-center">INP</text>
 <text x="14.732" y="10.795" size="1.016" layer="21" font="vector" ratio="15" rot="R270" align="bottom-center">REG</text>
-<text x="-2.794" y="1.778" size="1.4224" layer="21" font="vector" ratio="15" rot="R90" align="bottom-center">BLE Mate</text>
+<text x="-2.794" y="1.778" size="1.4224" layer="21" font="vector" ratio="15" rot="R90" align="bottom-center">BLE Mate2</text>
 <text x="10.795" y="17.653" size="1.016" layer="21" font="vector" ratio="15" rot="R90" align="bottom-center">LED1</text>
 <text x="7.747" y="17.653" size="1.016" layer="21" font="vector" ratio="15" rot="R90" align="bottom-center">LED0</text>
 <text x="-4.191" y="-0.635" size="1.6764" layer="16" font="vector" ratio="15" rot="MR90" align="bottom-center">V10</text>
 <text x="-45.72" y="24.13" size="1.778" layer="51" font="vector" ratio="15" align="bottom-center">M. Hord</text>
-<text x="7.366" y="38.354" size="1.778" layer="22" font="vector" ratio="15" rot="MR0" align="bottom-center">Keep this area
+<text x="7.366" y="38.354" size="1.778" layer="51" font="vector" ratio="15" rot="MR0" align="bottom-center">Keep this area
 clear of metal!</text>
 <text x="17.78" y="29.21" size="1.016" layer="22" font="vector" ratio="15" rot="MR90" align="top-center">P5</text>
@@
 <text x="17.78" y="11.43" size="0.8128" layer="22" font="vector" ratio="15" rot="MR90" align="top-center">VDD</text>
 <text x="17.78" y="8.763" size="0.8128" layer="22" font="vector" ratio="15" rot="MR90" align="top-center">GND</text>
-<text x="10.287" y="5.461" size="1.4224" layer="22" font="vector" ratio="15" rot="MR0" align="bottom-center">BLE Mate</text>
+<text x="10.414" y="5.461" size="1.4224" layer="22" font="vector" ratio="15" rot="MR0" align="bottom-center">BLE Mate2</text>
 <text x="-2.413" y="29.21" size="1.016" layer="22" font="vector" ratio="15" rot="MR90" align="bottom-center">A2</text>
 <text x="-2.413" y="26.67" size="1.016" layer="22" font="vector" ratio="15" rot="MR90" align="bottom-center">A1</text>
@@
 <attribute name="PROD_ID" value="RES-07828" x="48.26" y="-31.75" size="1.778" layer="27" display="off"/>
 </element>
-<element name="R6" library="SparkFun-Resistors" package="0603-RES" value="26.7k" x="12.065" y="6.35" rot="R90">
-<attribute name="PROD_ID" value="RES-12186" x="65.405" y="25.4" size="1.778" layer="27" rot="R90" display="off"/>
-</element>
-<element name="R7" library="SparkFun-Resistors" package="0603-RES" value="16.2k" x="13.589" y="6.35" rot="R90">
+<element name="R6" library="SparkFun-Resistors" package="0603-RES" value="16.2k" x="12.065" y="6.35" rot="R90">
+<attribute name="PROD_ID" value="RES-12187" x="65.405" y="25.4" size="1.778" layer="27" rot="R90" display="off"/>
+</element>
+<element name="R7" library="SparkFun-Resistors" package="0603-RES" value="26.7k" x="13.589" y="6.35" rot="R90">
 <attribute name="PROD_ID" value="RES-12187" x="66.929" y="29.21" size="1.778" layer="27" rot="R90" display="off"/>
 </element>
@@
 <attribute name="PROD_ID" value="CAP-00868" x="5.842" y="5.588" size="1.778" layer="27" font="vector" ratio="15" rot="R90" display="off"/>
 </element>
-<element name="LOGO1" library="SparkFun-Aesthetics" package="SFE_LOGO_NAME_.1" value="SFE_LOGO_NAME.1_INCH" x="20.32" y="-3.81" rot="R90"/>
+<element name="LOGO1" library="SparkFun-Aesthetics" package="SFE_LOGO_NAME_.1" value="SFE_LOGO_NAME.1_INCH" x="20.574" y="-4.191" rot="R90"/>
 <element name="LOGO2" library="SparkFun-Aesthetics" package="OSHW-LOGO-S" value="OSHW-LOGOS" x="-2.54" y="40.386"/>
-<element name="LOGO3" library="SparkFun-Aesthetics" package="SFE_LOGO_NAME_.1" value="SFE_LOGO_NAME.1_INCH" x="11.557" y="32.512" rot="MR0"/>
+<element name="LOGO3" library="SparkFun-Aesthetics" package="SFE_LOGO_NAME_FLAME_.1" value="SFE_LOGO_NAME_FLAME.1_INCH" x="12.319" y="32.893" rot="MR0"/>
 <element name="LOGO4" library="SparkFun-Aesthetics" package="OSHW-LOGO-S" value="OSHW-LOGOS" x="-2.159" y="33.02" rot="MR0"/>
 <element name="JP4" library="SparkFun-Connectors" package="1X06" value="" x="13.97" y="-5.08" rot="R180"/>
