File: Hardware/BC118_Mate.sch (EAGLE design)
At the start: 27 parts, among them Q1 BSS138, U2 AP2202-ADJ

Commit message: V01 ready for protos
Parts:
- added JP4: (no value), SparkFun-Connectors:M06SIP
Connections:
- new net CTS: JP1.5, JP4.5
- new net DTR: JP1.1, JP4.1
- net GND: now also JP4.6
- net RXI: now also JP4.2
- net TXO: now also JP4.3
- net VIN: now also JP4.4
Other:
- moved on the sheet: JP1
Changed lines of the file:
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@@
 <part name="LOGO3" library="SparkFun-Aesthetics" deviceset="SFE_LOGO_NAME" device=".1_INCH"/>
 <part name="LOGO4" library="SparkFun-Aesthetics" deviceset="OSHW-LOGO" device="S"/>
+<part name="JP4" library="SparkFun-Connectors" deviceset="M06" device="SIP"/>
 </parts>
 <sheets>
@@
 <attribute name="NAME" x="50.8" y="37.846" size="1.778" layer="95"/>
 </instance>
-<instance part="JP1" gate="G$1" x="233.68" y="162.56" rot="R180"/>
+<instance part="JP1" gate="G$1" x="241.3" y="162.56" rot="R180"/>
 <instance part="SUPPLY3" gate="G$1" x="45.72" y="38.1"/>
 <instance part="GND2" gate="1" x="17.78" y="10.16"/>
@@
 <instance part="SUPPLY8" gate="G$1" x="68.58" y="175.26"/>
 <instance part="GND6" gate="1" x="55.88" y="157.48"/>
-<instance part="GND7" gate="1" x="226.06" y="129.54"/>
+<instance part="GND7" gate="1" x="226.06" y="127"/>
 <instance part="LOGO1" gate="G$1" x="88.9" y="20.32"/>
 <instance part="LOGO2" gate="G$1" x="132.08" y="15.24"/>
 <instance part="LOGO3" gate="G$1" x="88.9" y="20.32"/>
 <instance part="LOGO4" gate="G$1" x="132.08" y="15.24"/>
+<instance part="JP4" gate="G$1" x="241.3" y="139.7" rot="R180"/>
 </instances>
 <busses>
@@
 <segment>
 <pinref part="JP1" gate="G$1" pin="3"/>
-<wire x1="228.6" y1="162.56" x2="223.52" y2="162.56" width="0.1524" layer="91"/>
+<wire x1="236.22" y1="162.56" x2="223.52" y2="162.56" width="0.1524" layer="91"/>
 <label x="220.98" y="162.56" size="1.27" layer="95" rot="R180" xref="yes"/>
 <pinref part="Q1" gate="G$1" pin="D"/>
@@
 <junction x="223.52" y="162.56"/>
 </segment>
+<segment>
+<pinref part="JP4" gate="G$1" pin="3"/>
+<wire x1="236.22" y1="139.7" x2="233.68" y2="139.7" width="0.1524" layer="91"/>
+<label x="233.68" y="139.7" size="1.27" layer="95" rot="R180" xref="yes"/>
+</segment>
 </net>
 <net name="RXI" class="0">
 <segment>
 <pinref part="JP1" gate="G$1" pin="2"/>
-<wire x1="228.6" y1="165.1" x2="220.98" y2="165.1" width="0.1524" layer="91"/>
+<wire x1="236.22" y1="165.1" x2="220.98" y2="165.1" width="0.1524" layer="91"/>
 <label x="220.98" y="165.1" size="1.27" layer="95" rot="R180" xref="yes"/>
 </segment>
@@
 <wire x1="200.66" y1="121.92" x2="203.2" y2="121.92" width="0.1524" layer="91"/>
 <label x="203.2" y="121.92" size="1.27" layer="95" xref="yes"/>
+</segment>
+<segment>
+<pinref part="JP4" gate="G$1" pin="2"/>
+<wire x1="236.22" y1="142.24" x2="233.68" y2="142.24" width="0.1524" layer="91"/>
+<label x="233.68" y="142.24" size="1.27" layer="95" rot="R180" xref="yes"/>
 </segment>
 </net>
@@
 <segment>
 <pinref part="JP1" gate="G$1" pin="6"/>
-<wire x1="226.06" y1="154.94" x2="228.6" y2="154.94" width="0.1524" layer="91"/>
+<wire x1="226.06" y1="154.94" x2="236.22" y2="154.94" width="0.1524" layer="91"/>
 <pinref part="GND7" gate="1" pin="GND"/>
+<wire x1="226.06" y1="129.54" x2="226.06" y2="132.08" width="0.1524" layer="91"/>
+<pinref part="JP4" gate="G$1" pin="6"/>
 <wire x1="226.06" y1="132.08" x2="226.06" y2="154.94" width="0.1524" layer="91"/>
+<wire x1="236.22" y1="132.08" x2="226.06" y2="132.08" width="0.1524" layer="91"/>
+<junction x="226.06" y="132.08"/>
 </segment>
 </net>
@@
 <wire x1="208.28" y1="160.02" x2="210.82" y2="160.02" width="0.1524" layer="91"/>
 <wire x1="210.82" y1="160.02" x2="218.44" y2="160.02" width="0.1524" layer="91"/>
-<wire x1="218.44" y1="160.02" x2="228.6" y2="160.02" width="0.1524" layer="91"/>
+<wire x1="218.44" y1="160.02" x2="236.22" y2="160.02" width="0.1524" layer="91"/>
 <wire x1="218.44" y1="147.32" x2="218.44" y2="160.02" width="0.1524" layer="91"/>
 <junction x="218.44" y="160.02"/>
@@
 <wire x1="210.82" y1="167.64" x2="210.82" y2="160.02" width="0.1524" layer="91"/>
 <junction x="210.82" y="160.02"/>
+</segment>
+<segment>
+<pinref part="JP4" gate="G$1" pin="4"/>
+<wire x1="236.22" y1="137.16" x2="233.68" y2="137.16" width="0.1524" layer="91"/>
+<label x="233.68" y="137.16" size="1.27" layer="95" rot="R180" xref="yes"/>
 </segment>
 </net>
@@
 <junction x="104.14" y="86.36"/>
 <pinref part="JP3" gate="G$1" pin="6"/>
+<label x="127" y="86.36" size="1.778" layer="95"/>
 </segment>
 </net>
@@
 <pinref part="JP3" gate="G$1" pin="5"/>
 <wire x1="119.38" y1="88.9" x2="134.62" y2="88.9" width="0.1524" layer="91"/>
+<label x="127" y="88.9" size="1.778" layer="95"/>
 </segment>
 </net>
@@
 <pinref part="JP3" gate="G$1" pin="3"/>
 <wire x1="96.52" y1="93.98" x2="134.62" y2="93.98" width="0.1524" layer="91"/>
+<label x="127" y="93.98" size="1.778" layer="95"/>
 </segment>
 </net>
@@
 <pinref part="JP3" gate="G$1" pin="2"/>
 <wire x1="96.52" y1="96.52" x2="134.62" y2="96.52" width="0.1524" layer="91"/>
+<label x="127" y="96.52" size="1.778" layer="95"/>
 </segment>
 </net>
@@
 <pinref part="JP3" gate="G$1" pin="1"/>
 <wire x1="96.52" y1="99.06" x2="134.62" y2="99.06" width="0.1524" layer="91"/>
+<label x="127" y="99.06" size="1.778" layer="95"/>
 </segment>
 </net>
@@
 <wire x1="124.46" y1="121.92" x2="134.62" y2="121.92" width="0.1524" layer="91"/>
 <wire x1="104.14" y1="101.6" x2="124.46" y2="121.92" width="0.1524" layer="91"/>
+<label x="127" y="121.92" size="1.778" layer="95"/>
 </segment>
 </net>
@@
 <wire x1="124.46" y1="124.46" x2="134.62" y2="124.46" width="0.1524" layer="91"/>
 <wire x1="104.14" y1="104.14" x2="124.46" y2="124.46" width="0.1524" layer="91"/>
+<label x="127" y="124.46" size="1.778" layer="95"/>
 </segment>
 </net>
@@
 <pinref part="JP2" gate="G$1" pin="1"/>
 <wire x1="124.46" y1="132.08" x2="134.62" y2="132.08" width="0.1524" layer="91"/>
+<label x="127" y="132.08" size="1.778" layer="95"/>
 </segment>
 </net>
@@
 <pinref part="JP2" gate="G$1" pin="2"/>
 <wire x1="124.46" y1="129.54" x2="134.62" y2="129.54" width="0.1524" layer="91"/>
+<label x="127" y="129.54" size="1.778" layer="95"/>
 </segment>
 </net>
@@
 <pinref part="JP2" gate="G$1" pin="3"/>
 <wire x1="116.84" y1="127" x2="134.62" y2="127" width="0.1524" layer="91"/>
+<label x="127" y="127" size="1.778" layer="95"/>
 </segment>
 </net>
@@
 <pinref part="U1" gate="G2" pin="PIO_2"/>
 <wire x1="121.92" y1="106.68" x2="96.52" y2="106.68" width="0.1524" layer="91"/>
+<label x="127" y="83.82" size="1.778" layer="95"/>
 </segment>
 </net>
@@
 <pinref part="JP3" gate="G$1" pin="4"/>
 <wire x1="116.84" y1="91.44" x2="134.62" y2="91.44" width="0.1524" layer="91"/>
+<label x="127" y="91.44" size="1.778" layer="95"/>
 </segment>
 </net>
@@
 <wire x1="124.46" y1="119.38" x2="134.62" y2="119.38" width="0.1524" layer="91"/>
 <wire x1="106.68" y1="101.6" x2="124.46" y2="119.38" width="0.1524" layer="91"/>
-</segment>
-</net>
+<label x="127" y="119.38" size="1.778" layer="95"/>
+</segment>
+</net>
+<net name="DTR" class="0">
+<segment>
+<pinref part="JP1" gate="G$1" pin="1"/>
+<wire x1="236.22" y1="167.64" x2="233.68" y2="167.64" width="0.1524" layer="91"/>
+<label x="233.68" y="167.64" size="1.27" layer="95" rot="R180" xref="yes"/>
+</segment>
+<segment>
+<pinref part="JP4" gate="G$1" pin="1"/>
+<wire x1="236.22" y1="144.78" x2="233.68" y2="144.78" width="0.1524" layer="91"/>
+<label x="233.68" y="144.78" size="1.27" layer="95" rot="R180" xref="yes"/>
+</segment>
+</net>
+<net name="CTS" class="0">
+<segment>
+<pinref part="JP1" gate="G$1" pin="5"/>
+<wire x1="236.22" y1="157.48" x2="233.68" y2="157.48" width="0.1524" layer="91"/>
+<label x="233.68" y="157.48" size="1.27" layer="95" rot="R180" xref="yes"/>
+</segment>
+<segment>
+<pinref part="JP4" gate="G$1" pin="5"/>
+<wire x1="236.22" y1="134.62" x2="233.68" y2="134.62" width="0.1524" layer="91"/>
+<label x="233.68" y="134.62" size="1.27" layer="95" rot="R180" xref="yes"/>
+</segment>
+</net>
