File: Hardware/BC118_Mate.sch (EAGLE design)
At the start: 28 parts, among them Q1 BSS138, U2 AP2202-ADJ

Commit message: Change LED pin assignments to match new firmware
Parts:
- LED0: value RED -> BLUE; device SparkFun-LED:LED-RED0603 -> SparkFun-LED:LED-BLUE0603
- LED1: value BLUE -> RED; device SparkFun-LED:LED-BLUE0603 -> SparkFun-LED:LED-RED0603
Connections:
- net N$8: now also LED0.C; no longer LED1.C
- net N$9: now also LED1.C; no longer LED0.C
- net PIO_10: no longer LED1.A
- net PIO_4: now also LED0.A
- net PIO_9: now also LED1.A; no longer LED0.A
Other:
- note added: "v10"
- note removed: "v01"
- moved on the sheet: LED0, LED1
Changed lines of the file:
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@@
 <layer number="254" name="cooling" color="7" fill="1" visible="yes" active="yes"/>
 </layers>
-<schematic xreflabel="%F%N/%S.%C%R" xrefpart="1_/%S.%C%R">
+<schematic xreflabel="%F%N/%S" xrefpart="1_/%S.%C%R">
 <attributes>
 </attributes>
@@
 <part name="R5" library="SparkFun-Resistors" deviceset="1KOHM1/10W1%(0603)" device="" value="1K"/>
 <part name="R8" library="SparkFun-Resistors" deviceset="1KOHM1/10W1%(0603)" device="" value="1K"/>
-<part name="LED1" library="SparkFun-LED" deviceset="LED-BLUE" device="0603" value="BLUE"/>
-<part name="LED0" library="SparkFun-LED" deviceset="LED-RED" device="0603" value="RED"/>
+<part name="LED0" library="SparkFun-LED" deviceset="LED-BLUE" device="0603" value="BLUE"/>
+<part name="LED1" library="SparkFun-LED" deviceset="LED-RED" device="0603" value="RED"/>
 <part name="LEDS" library="SparkFun-Passives" deviceset="JUMPER-PAD-3-NC_BY_PASTE" device=""/>
 <part name="GND4" library="SparkFun-Aesthetics" deviceset="GND" device=""/>
@@
 for minimal power use, as well, but that's your problem!</text>
 <text x="167.64" y="7.62" size="3.81" layer="94">M. Hord</text>
-<text x="238.252" y="7.366" size="3.81" layer="94">v01</text>
+<text x="238.252" y="7.366" size="3.81" layer="94">v10</text>
 </plain>
 <instances>
@@
 <instance part="R5" gate="G$1" x="119.38" y="63.5" rot="R90"/>
 <instance part="R8" gate="G$1" x="104.14" y="63.5" rot="R90"/>
-<instance part="LED1" gate="G$1" x="104.14" y="76.2"/>
-<instance part="LED0" gate="G$1" x="119.38" y="76.2"/>
+<instance part="LED0" gate="G$1" x="104.14" y="76.2"/>
+<instance part="LED1" gate="G$1" x="119.38" y="76.2"/>
 <instance part="LEDS" gate="G$1" x="111.76" y="53.34" smashed="yes" rot="R90">
 <attribute name="NAME" x="108.712" y="55.245" size="1.778" layer="95"/>
@@
 <segment>
 <pinref part="R8" gate="G$1" pin="2"/>
+<pinref part="LED0" gate="G$1" pin="C"/>
+<wire x1="104.14" y1="68.58" x2="104.14" y2="71.12" width="0.1524" layer="91"/>
+</segment>
+</net>
+<net name="N$9" class="0">
+<segment>
+<pinref part="R5" gate="G$1" pin="2"/>
 <pinref part="LED1" gate="G$1" pin="C"/>
-<wire x1="104.14" y1="68.58" x2="104.14" y2="71.12" width="0.1524" layer="91"/>
-</segment>
-</net>
-<net name="N$9" class="0">
-<segment>
-<pinref part="R5" gate="G$1" pin="2"/>
-<pinref part="LED0" gate="G$1" pin="C"/>
 <wire x1="119.38" y1="68.58" x2="119.38" y2="71.12" width="0.1524" layer="91"/>
 </segment>
@@
 <net name="PIO_10" class="0">
 <segment>
-<pinref part="LED1" gate="G$1" pin="A"/>
-<wire x1="104.14" y1="78.74" x2="104.14" y2="86.36" width="0.1524" layer="91"/>
 <pinref part="U1" gate="G2" pin="PIO_10"/>
-<wire x1="104.14" y1="86.36" x2="96.52" y2="86.36" width="0.1524" layer="91"/>
-<wire x1="104.14" y1="86.36" x2="134.62" y2="86.36" width="0.1524" layer="91"/>
-<junction x="104.14" y="86.36"/>
+<wire x1="96.52" y1="86.36" x2="134.62" y2="86.36" width="0.1524" layer="91"/>
 <pinref part="JP3" gate="G$1" pin="6"/>
 <label x="127" y="86.36" size="1.778" layer="95"/>
@@
 <net name="PIO_9" class="0">
 <segment>
-<pinref part="LED0" gate="G$1" pin="A"/>
+<pinref part="LED1" gate="G$1" pin="A"/>
 <wire x1="119.38" y1="78.74" x2="119.38" y2="88.9" width="0.1524" layer="91"/>
 <pinref part="U1" gate="G2" pin="PIO_9"/>
@@
 <wire x1="104.14" y1="101.6" x2="124.46" y2="121.92" width="0.1524" layer="91"/>
 <label x="127" y="121.92" size="1.778" layer="95"/>
-</segment>
-</net>
+<pinref part="LED0" gate="G$1" pin="A"/>
+<wire x1="104.14" y1="78.74" x2="104.14" y2="101.6" width="0.1524" layer="91"/>
+<junction x="104.14" y="101.6"/>
+</segment>
+</net>

Commit message: Ready for reds
Parts:
- LOGO3: value SFE_LOGO_NAME.1_INCH -> SFE_LOGO_NAME_FLAME.1_INCH; device SparkFun-Aesthetics:SFE_LOGO_NAME.1_INCH -> SparkFun-Aesthetics:SFE_LOGO_NAME_FLAME.1_INCH
- R6: value 26.7k -> 16.2k; device SparkFun-Resistors:26.7KOHM1/10W1%(0603) -> SparkFun-Resistors:16.2KOHM1/10W1%(0603)
- R7: value 16.2k -> 26.7k
Changed lines of the file:
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@@
 <part name="R4" library="SparkFun-Resistors" deviceset="10KOHM1/10W1%(0603)" device="0603" value="10K"/>
 <part name="R2" library="SparkFun-Resistors" deviceset="100KOHM1/10W1%(0603)" device="" value="100k"/>
-<part name="R6" library="SparkFun-Resistors" deviceset="26.7KOHM1/10W1%(0603)" device="" value="26.7k"/>
-<part name="R7" library="SparkFun-Resistors" deviceset="16.2KOHM1/10W1%(0603)" device="" value="16.2k"/>
+<part name="R6" library="SparkFun-Resistors" deviceset="16.2KOHM1/10W1%(0603)" device="" value="16.2k"/>
+<part name="R7" library="SparkFun-Resistors" deviceset="16.2KOHM1/10W1%(0603)" device="" value="26.7k"/>
 <part name="U2" library="SparkFun-PowerIC" deviceset="AP2202-ADJ" device="" value="AP2202-ADJ"/>
 <part name="INP" library="SparkFun-Passives" deviceset="JUMPER-PAD-3-2OF3_NC_BY_PASTE" device=""/>
@@
 <part name="LOGO1" library="SparkFun-Aesthetics" deviceset="SFE_LOGO_NAME" device=".1_INCH"/>
 <part name="LOGO2" library="SparkFun-Aesthetics" deviceset="OSHW-LOGO" device="S"/>
-<part name="LOGO3" library="SparkFun-Aesthetics" deviceset="SFE_LOGO_NAME" device=".1_INCH"/>
+<part name="LOGO3" library="SparkFun-Aesthetics" deviceset="SFE_LOGO_NAME_FLAME" device=".1_INCH"/>
 <part name="LOGO4" library="SparkFun-Aesthetics" deviceset="OSHW-LOGO" device="S"/>
 <part name="JP4" library="SparkFun-Connectors" deviceset="M06" device="SIP"/>
@@
 <instance part="GND6" gate="1" x="55.88" y="157.48"/>
 <instance part="GND7" gate="1" x="226.06" y="127"/>
-<instance part="LOGO1" gate="G$1" x="88.9" y="20.32"/>
+<instance part="LOGO1" gate="G$1" x="87.376" y="19.304"/>
 <instance part="LOGO2" gate="G$1" x="132.08" y="15.24"/>
-<instance part="LOGO3" gate="G$1" x="88.9" y="20.32"/>
+<instance part="LOGO3" gate="G$1" x="88.646" y="19.05"/>
 <instance part="LOGO4" gate="G$1" x="132.08" y="15.24"/>
 <instance part="JP4" gate="G$1" x="241.3" y="139.7" rot="R180"/>
