File: Hardware/BLE_Mate2.sch (EAGLE design)
At the start: 28 parts, among them Q1 BSS138, U2 AP2202-ADJ

Commit message: added board fiducials
Parts:
- added FID1, FID2: FIDUCIAL1X2, SparkFun-Aesthetics:FIDUCIAL1X2
Changed lines of the file:
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@@
 <?xml version="1.0" encoding="utf-8"?>
 <!DOCTYPE eagle SYSTEM "eagle.dtd">
-<eagle version="6.5.0">
+<eagle version="6.6.0">
 <drawing>
 <settings>
@@
 <part name="LOGO4" library="SparkFun-Aesthetics" deviceset="OSHW-LOGO" device="S"/>
 <part name="JP4" library="SparkFun-Connectors" deviceset="M06" device="SIP"/>
+<part name="FID1" library="SparkFun-Aesthetics" deviceset="FIDUCIAL" device="1X2"/>
+<part name="FID2" library="SparkFun-Aesthetics" deviceset="FIDUCIAL" device="1X2"/>
 </parts>
 <sheets>
@@
 <instance part="LOGO4" gate="G$1" x="132.08" y="15.24"/>
 <instance part="JP4" gate="G$1" x="241.3" y="139.7" rot="R180"/>
+<instance part="FID1" gate="G$1" x="238.76" y="33.02"/>
+<instance part="FID2" gate="G$1" x="246.38" y="33.02"/>
 </instances>
 <busses>
